Commit message: remove world link from urdf (and others)

File: tra1_description/urdf/tra1.xacro (robot description, xacro)
@@ -27,10 +27,4 @@
   <xacro:property name="J5Y_J6Y" value="-0.05"/>
   <xacro:property name="J5Z_J6Z" value="1.3795"/>
-  <!-- Used for fixing robot to Gazebo 'base_link' -->
-  <link name="world"/>
-  <joint name="fixed" type="fixed">
-    <parent link="world"/>
-    <child link="base_link"/>
-  </joint>
   <!-- ==================================================================base_link -->
   <link name="base_link">

Commit message: add limit tag, change joint type from continuous to revolute

File: tra1_description/urdf/tra1.xacro (robot description, xacro)
@@ -45,5 +45,5 @@
   </link>
   <!-- +++++++++++++++++++++++++++++++++++++++++++++++++++++++++++++++++joint1 -->
-  <joint name="joint1" type="continuous">
+  <joint name="joint1" type="revolute">
     <parent link="base_link"/>
     <child link="link_j1"/>
@@ -51,4 +51,5 @@
     <axis xyz="0 0 1"/>
     <dynamics damping="0.7"/>
+    <limit upper="2.18" lower="-2.18" effort="10" velocity="1" />
   </joint>
   <!-- ==================================================================link1 -->
@@ -63,5 +64,5 @@
   </link>
   <!-- +++++++++++++++++++++++++++++++++++++++++++++++++++++++++++++++++joint2 -->
-  <joint name="joint2" type="continuous">
+  <joint name="joint2" type="revolute">
     <parent link="link_j1"/>
     <child link="link_j2"/>
@@ -69,4 +70,5 @@
     <axis xyz="1 0 0"/>
     <dynamics damping="0.7"/>
+    <limit upper="2.18" lower="-2.18" effort="10" velocity="1" />
   </joint>
   <!-- ==================================================================link2 -->
@@ -81,5 +83,5 @@
   </link>
   <!-- +++++++++++++++++++++++++++++++++++++++++++++++++++++++++++++++++joint3 -->
-    <joint name="joint3" type="continuous">
+    <joint name="joint3" type="revolute">
       <parent link="link_j2"/>
       <child link="link_j3"/>
@@ -87,4 +89,5 @@
       <axis xyz="1 0 0"/>
       <dynamics damping="0.7"/>
+      <limit upper="2.18" lower="-2.18" effort="10" velocity="1" />
     </joint>
   <!-- ==================================================================link3 -->
@@ -99,5 +102,5 @@
   </link>
   <!-- +++++++++++++++++++++++++++++++++++++++++++++++++++++++++++++++++joint4 -->
-  <joint name="joint4" type="continuous">
+  <joint name="joint4" type="revolute">
     <parent link="link_j3"/>
     <child link="link_j4"/>
@@ -105,4 +108,5 @@
     <axis xyz="0 0 1"/>
     <dynamics damping="0.7"/>
+    <limit upper="2.18" lower="-2.18" effort="10" velocity="1" />
   </joint>
   <!-- ==================================================================link4 -->
@@ -117,5 +121,5 @@
   </link>
   <!-- +++++++++++++++++++++++++++++++++++++++++++++++++++++++++++++++++joint5 -->
-  <joint name="joint5" type="continuous">
+  <joint name="joint5" type="revolute">
     <parent link="link_j4"/>
     <child link="link_j5"/>
@@ -123,4 +127,5 @@
     <axis xyz="1 0 0"/>
     <dynamics damping="0.7"/>
+    <limit upper="2.18" lower="-2.18" effort="10" velocity="1" />
   </joint>
   <!-- ==================================================================link5 -->
@@ -135,5 +140,5 @@
   </link>
   <!-- +++++++++++++++++++++++++++++++++++++++++++++++++++++++++++++++++joint6 -->
-  <joint name="joint6" type="continuous">
+  <joint name="joint6" type="revolute">
     <parent link="link_j5"/>
     <child link="link_j6"/>
@@ -141,4 +146,5 @@
     <axis xyz="0 0 1"/>
     <dynamics damping="0.7"/>
+    <limit upper="2.18" lower="-2.18" effort="10" velocity="1" />
   </joint>
   <!-- ==================================================================link6 -->
