Commit message: Change material color to improve the sight

File: tra1_description/urdf/materials.xacro (robot description, xacro)
@@ -24,6 +24,30 @@
     <color rgba="0.0 0.8 0.0 1.0"/>
   </material>
-  <material name="grey">
+  <material name="grey1">
+    <color rgba="0.1 0.1 0.1 1.0"/>
+  </material>
+  <material name="grey2">
     <color rgba="0.2 0.2 0.2 1.0"/>
+  </material>
+  <material name="grey3">
+    <color rgba="0.3 0.3 0.3 1.0"/>
+  </material>
+  <material name="grey4">
+    <color rgba="0.4 0.4 0.4 1.0"/>
+  </material>
+  <material name="grey5">
+    <color rgba="0.5 0.5 0.5 1.0"/>
+  </material>
+  <material name="grey6">
+    <color rgba="0.6 0.6 0.6 1.0"/>
+  </material>
+  <material name="grey7">
+    <color rgba="0.7 0.7 0.7 1.0"/>
+  </material>
+  <material name="grey8">
+    <color rgba="0.8 0.8 0.8 1.0"/>
+  </material>
+  <material name="grey9">
+    <color rgba="0.9 0.9 0.9 1.0"/>
   </material>
   <material name="orange">

File: tra1_description/urdf/tra1.xacro (robot description, xacro)
@@ -49,5 +49,5 @@
             <mesh filename="package://tra1_description/meshes/B.STL" scale="${MODEL_RATIO} ${MODEL_RATIO} ${MODEL_RATIO}"/>
         </geometry>
-        <material name="grey"/>
+        <material name="grey4"/>
     </visual>
   </link>
@@ -68,5 +68,5 @@
         <mesh filename="package://tra1_description/meshes/J1.STL" scale="${MODEL_RATIO} ${MODEL_RATIO} ${MODEL_RATIO}"/>
       </geometry>
-      <material name="black"/>
+      <material name="grey6"/>
     </visual>
   </link>
@@ -87,5 +87,5 @@
         <mesh filename="package://tra1_description/meshes/J2.STL" scale="${MODEL_RATIO} ${MODEL_RATIO} ${MODEL_RATIO}"/>
       </geometry>
-      <material name="grey"/>
+      <material name="grey4"/>
     </visual>
   </link>
@@ -106,5 +106,5 @@
         <mesh filename="package://tra1_description/meshes/J3.STL" scale="${MODEL_RATIO} ${MODEL_RATIO} ${MODEL_RATIO}"/>
       </geometry>
-      <material name="grey"/>
+      <material name="grey6"/>
     </visual>
   </link>
@@ -125,5 +125,5 @@
         <mesh filename="package://tra1_description/meshes/J4.STL" scale="${MODEL_RATIO} ${MODEL_RATIO} ${MODEL_RATIO}"/>
       </geometry>
-      <material name="black"/>
+      <material name="grey4"/>
     </visual>
   </link>
@@ -144,5 +144,5 @@
         <mesh filename="package://tra1_description/meshes/J5.STL" scale="${MODEL_RATIO} ${MODEL_RATIO} ${MODEL_RATIO}"/>
       </geometry>
-      <material name="grey"/>
+      <material name="grey6"/>
     </visual>
   </link>
@@ -163,5 +163,5 @@
         <mesh filename="package://tra1_description/meshes/J6.STL" scale="${MODEL_RATIO} ${MODEL_RATIO} ${MODEL_RATIO}"/>
       </geometry>
-      <material name="black"/>
+      <material name="grey4"/>
     </visual>
   </link>
